File: hardware/photodiode-opamp-tester-mk-1.0.brd (EAGLE design)
At the start: 25.4 x 15.2 mm, 15 parts, among them U1 MCP6001

Commit message: more photodiode dickery
Routing:
- net N$3: track 0.00 -> 54.9 mm, vias 0 -> 1
- net N$2: track 0.00 -> 19.2 mm, vias 0 -> 1
- net VCC: track 0.00 -> 7.75 mm
- net OUT: track 0.00 -> 7.35 mm
Other:
- outline, holes or cut-outs redrawn
Changed lines of the file:
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@@
 <board>
 <plain>
-<wire x1="0" y1="15.24" x2="25.4" y2="15.24" width="0" layer="20"/>
-<wire x1="25.4" y1="15.24" x2="25.4" y2="0" width="0" layer="20"/>
-<wire x1="25.4" y1="0" x2="0" y2="0" width="0" layer="20"/>
-<wire x1="0" y1="0" x2="0" y2="15.24" width="0" layer="20"/>
+<wire x1="1.905" y1="15.24" x2="23.495" y2="15.24" width="0" layer="20"/>
+<wire x1="23.495" y1="15.24" x2="25.4" y2="13.335" width="0" layer="20" curve="-90"/>
+<wire x1="25.4" y1="13.335" x2="25.4" y2="1.905" width="0" layer="20"/>
+<wire x1="25.4" y1="1.905" x2="23.495" y2="0" width="0" layer="20" curve="-90"/>
+<wire x1="23.495" y1="0" x2="1.905" y2="0" width="0" layer="20"/>
+<wire x1="1.905" y1="0" x2="0" y2="1.905" width="0" layer="20" curve="-90"/>
+<wire x1="0" y1="1.905" x2="0" y2="13.335" width="0" layer="20"/>
+<wire x1="0" y1="13.335" x2="1.905" y2="15.24" width="0" layer="20" curve="-90"/>
 <text x="19.685" y="6.35" size="0.8" layer="21" font="vector" ratio="10" rot="SR0" align="center">&gt;VERSION</text>
 <text x="11.43" y="7.62" size="1.016" layer="22" font="vector" ratio="16" rot="MR270" align="center">&gt;VERSION</text>
@@
 <signal name="GND">
 <polygon width="0.1524" layer="1" rank="6">
-<vertex x="0" y="15.24"/>
-<vertex x="25.4" y="15.24"/>
-<vertex x="25.4" y="0"/>
-<vertex x="0" y="0"/>
+<vertex x="1.905" y="15.24"/>
+<vertex x="23.495" y="15.24" curve="-90"/>
+<vertex x="25.4" y="13.335"/>
+<vertex x="25.4" y="1.905" curve="-90"/>
+<vertex x="23.495" y="0"/>
+<vertex x="1.905" y="0" curve="-90"/>
+<vertex x="0" y="1.905"/>
+<vertex x="0" y="13.335" curve="-90"/>
 </polygon>
 <contactref element="JP1" pad="1"/>
@@
 <contactref element="U1" pad="1"/>
 <contactref element="R1" pad="S"/>
-<wire x1="4.7" y1="3.81" x2="5.4" y2="7.5899" width="0" layer="19" extent="1-1"/>
-<wire x1="1.27" y1="5.08" x2="4.7" y2="3.81" width="0" layer="19" extent="1-1"/>
+<wire x1="5.4" y1="7.5899" x2="5.4" y2="6.67" width="0.3048" layer="1"/>
+<wire x1="5.4" y1="6.67" x2="3.81" y2="5.08" width="0.3048" layer="1"/>
+<wire x1="3.81" y1="5.08" x2="1.27" y2="5.08" width="0.3048" layer="1"/>
+<wire x1="4.7" y1="3.81" x2="4.7" y2="4.19" width="0.3048" layer="1"/>
+<wire x1="4.7" y1="4.19" x2="3.81" y2="5.08" width="0.3048" layer="1"/>
 </signal>
 <signal name="VCC">
@@
 <contactref element="C1" pad="1"/>
 <contactref element="U1" pad="5"/>
-<wire x1="5.4" y1="10.1901" x2="5.5" y2="12.7" width="0" layer="19" extent="1-1"/>
-<wire x1="1.27" y1="7.62" x2="5.4" y2="10.1901" width="0" layer="19" extent="1-1"/>
+<wire x1="1.27" y1="7.62" x2="2.8299" y2="7.62" width="0.3048" layer="1"/>
+<wire x1="2.8299" y1="7.62" x2="5.4" y2="10.1901" width="0.3048" layer="1"/>
+<wire x1="5.5" y1="12.7" x2="5.5" y2="10.2901" width="0.3048" layer="1"/>
+<wire x1="5.5" y1="10.2901" x2="5.4" y2="10.1901" width="0.3048" layer="1"/>
 </signal>
 <signal name="N$2">
@@
 <contactref element="R1" pad="E"/>
 <contactref element="TP1" pad="1"/>
-<wire x1="10.16" y1="10.58" x2="12.7" y2="10.58" width="0" layer="19" extent="1-1"/>
-<wire x1="8.1" y1="5.01" x2="10.16" y2="10.58" width="0" layer="19" extent="1-1"/>
-<wire x1="1.27" y1="10.16" x2="8.1" y2="5.01" width="0" layer="19" extent="1-1"/>
+<wire x1="12.7" y1="10.58" x2="10.16" y2="10.58" width="0.3048" layer="1"/>
+<wire x1="10.16" y1="10.58" x2="10.16" y2="6.985" width="0.3048" layer="1"/>
+<via x="10.16" y="6.985" extent="1-16" drill="0.3302"/>
+<wire x1="10.16" y1="6.985" x2="8.255" y2="6.985" width="0.3048" layer="16"/>
+<wire x1="8.255" y1="6.985" x2="5.08" y2="10.16" width="0.3048" layer="16"/>
+<wire x1="5.08" y1="10.16" x2="1.27" y2="10.16" width="0.3048" layer="16"/>
+<wire x1="8.1" y1="5.01" x2="8.185" y2="5.01" width="0.3048" layer="1"/>
+<wire x1="8.185" y1="5.01" x2="10.16" y2="6.985" width="0.3048" layer="1"/>
 </signal>
 <signal name="N$3">
@@
 <contactref element="PD6" pad="K"/>
 <contactref element="PD5" pad="K"/>
-<wire x1="20.105" y1="10.795" x2="19.955" y2="13.335" width="0" layer="19" extent="1-1"/>
-<wire x1="15.875" y1="12.93" x2="19.955" y2="13.335" width="0" layer="19" extent="1-1"/>
-<wire x1="12.7" y1="12.28" x2="15.875" y2="12.93" width="0" layer="19" extent="1-1"/>
-<wire x1="10.16" y1="12.28" x2="12.7" y2="12.28" width="0" layer="19" extent="1-1"/>
-<wire x1="7.3" y1="10.1901" x2="10.16" y2="12.28" width="0" layer="19" extent="1-1"/>
-<wire x1="17.145" y1="4.445" x2="20.105" y2="10.795" width="0" layer="19" extent="1-1"/>
-<wire x1="12.065" y1="5.08" x2="17.145" y2="4.445" width="0" layer="19" extent="1-1"/>
-<wire x1="22.225" y1="4.675" x2="17.145" y2="4.445" width="0" layer="19" extent="1-1"/>
-<wire x1="1.27" y1="12.7" x2="7.3" y2="10.1901" width="0" layer="19" extent="1-1"/>
+<wire x1="7.3" y1="10.1901" x2="7.3" y2="10.475" width="0.3048" layer="1"/>
+<wire x1="7.3" y1="10.475" x2="9.105" y2="12.28" width="0.3048" layer="1"/>
+<wire x1="9.105" y1="12.28" x2="10.16" y2="12.28" width="0.3048" layer="1"/>
+<wire x1="10.16" y1="12.28" x2="12.7" y2="12.28" width="0.3048" layer="1"/>
+<wire x1="12.7" y1="12.28" x2="13.55" y2="12.28" width="0.3048" layer="1"/>
+<wire x1="13.55" y1="12.28" x2="14.2" y2="12.93" width="0.3048" layer="1"/>
+<wire x1="14.2" y1="12.93" x2="15.875" y2="12.93" width="0.3048" layer="1"/>
+<wire x1="15.875" y1="12.93" x2="17.375" y2="12.93" width="0.3048" layer="1"/>
+<wire x1="17.375" y1="12.93" x2="17.78" y2="13.335" width="0.3048" layer="1"/>
+<wire x1="17.78" y1="13.335" x2="19.955" y2="13.335" width="0.3048" layer="1"/>
+<wire x1="19.955" y1="13.335" x2="19.955" y2="10.945" width="0.3048" layer="1"/>
+<wire x1="19.955" y1="10.945" x2="20.105" y2="10.795" width="0.3048" layer="1"/>
+<wire x1="12.065" y1="5.08" x2="13.97" y2="5.08" width="0.3048" layer="1"/>
+<wire x1="13.97" y1="5.08" x2="17.78" y2="8.89" width="0.3048" layer="1"/>
+<wire x1="17.78" y1="8.89" x2="19.685" y2="10.795" width="0.3048" layer="1"/>
+<wire x1="17.145" y1="4.445" x2="16.51" y2="5.08" width="0.3048" layer="1"/>
+<wire x1="16.51" y1="5.08" x2="13.97" y2="5.08" width="0.3048" layer="1"/>
+<wire x1="19.685" y1="10.795" x2="20.105" y2="10.795" width="0.3048" layer="1"/>
+<wire x1="22.225" y1="4.675" x2="21.995" y2="4.675" width="0.3048" layer="1"/>
+<wire x1="21.995" y1="4.675" x2="17.78" y2="8.89" width="0.3048" layer="1"/>
+<via x="17.78" y="8.89" extent="1-16" drill="0.3302"/>
+<wire x1="1.27" y1="12.7" x2="13.97" y2="12.7" width="0.3048" layer="16"/>
+<wire x1="13.97" y1="12.7" x2="17.78" y2="8.89" width="0.3048" layer="16"/>
 </signal>
 </signals>
-<errors>
-</errors>
 </board>
 </drawing>
