File: hardware/tricorder-photodiode-breakout-mk-1.0.brd (EAGLE design)
At the start: 50.8 x 25.4 mm, 9 parts

Commit message: quad opamps
Parts:
- added C2: 100n, a_parts:C0603
- added PD7: SD019-141-411-IR, a_parts:LED-0805
- added U2: (no value), a_parts:SO14
- PD1: value GUVA-S12SD -> SD019-141-411-R; device a_parts:LED3528 -> a_parts:LED-0805
- PD2: value GUVB-S11SD -> SD019-141-411-G; device a_parts:LED3528 -> a_parts:LED-0805
- PD3: value SD019-141-411-R -> SD019-141-411-B
- PD4: value SD019-141-411-G -> SD019-111-411
- PD5: value SD019-141-411-B -> GUVA-S12SD; device a_parts:LED-0805 -> a_parts:LED3528
- PD6: value SD019-111-411 -> GUVB-S11SD; device a_parts:LED-0805 -> a_parts:LED3528
- U1: device a_parts:SO08 -> a_parts:SO14
- moved PD6 16.2 mm to (1.91, -12.1)
- moved PD5 11.5 mm to (1.91, -17.8)
- moved PD2 10.8 mm to (-6.35, -19.1)
- moved U1 7.65 mm to (-17.1, -24.8)
- moved PD3 6.35 mm to (-9.53, -19.1)
- moved PD4 6.35 mm to (-12.7, -19.1)
- moved PD1 5.24 mm to (-3.17, -19.1)
Connections:
- new net 3.3V: C1.1, C2.1, U1.4, U2.4
- new net GND: C1.2, C2.2, U1.11, U2.11
- new net INA+: U1.3
- new net INA-: U1.2
- new net INB+: U1.5
- new net INB-: U1.6
- new net INC+: U1.10
- new net INC-: U1.9
- new net IND+: U1.12
- new net IND-: U1.13
- new net INE+: U2.3
- new net INE-: U2.2
- new net INF+: U2.5
- new net INF-: U2.6
- new net ING+: U2.10
- new net ING-: U2.9
- new net INH+: U2.12
- new net INH-: U2.13
- new net OUTA: U1.1
- new net OUTB: U1.7
- new net OUTC: U1.8
- new net OUTD: U1.14
- new net OUTE: U2.1
- new net OUTF: U2.7
- new net OUTG: U2.8
- new net OUTH: U2.14
Changed lines of the file:
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@@
 </element>
 <element name="C1" library="a_parts" package="C0603" value="100n" x="8.255" y="15.875"/>
-<element name="PD2" library="a_parts" package="LED3528" value="GUVB-S11SD" x="1.905" y="-12.065"/>
-<element name="PD1" library="a_parts" package="LED3528" value="GUVA-S12SD" x="1.905" y="-17.78"/>
-<element name="PD3" library="a_parts" package="LED-0805" value="SD019-141-411-R" x="-3.175" y="-19.05"/>
-<element name="PD4" library="a_parts" package="LED-0805" value="SD019-141-411-G" x="-6.35" y="-19.05"/>
-<element name="PD5" library="a_parts" package="LED-0805" value="SD019-141-411-B" x="-9.525" y="-19.05"/>
-<element name="PD6" library="a_parts" package="LED-0805" value="SD019-111-411" x="-12.7" y="-19.05"/>
-<element name="U1" library="a_parts" package="SO08" value="" x="-16.51" y="-17.145"/>
+<element name="PD6" library="a_parts" package="LED3528" value="GUVB-S11SD" x="1.905" y="-12.065"/>
+<element name="PD5" library="a_parts" package="LED3528" value="GUVA-S12SD" x="1.905" y="-17.78"/>
+<element name="PD1" library="a_parts" package="LED-0805" value="SD019-141-411-R" x="-3.175" y="-19.05"/>
+<element name="PD2" library="a_parts" package="LED-0805" value="SD019-141-411-G" x="-6.35" y="-19.05"/>
+<element name="PD3" library="a_parts" package="LED-0805" value="SD019-141-411-B" x="-9.525" y="-19.05"/>
+<element name="PD4" library="a_parts" package="LED-0805" value="SD019-111-411" x="-12.7" y="-19.05"/>
+<element name="PD7" library="a_parts" package="LED-0805" value="SD019-141-411-IR" x="-21.59" y="-19.05"/>
+<element name="U1" library="a_parts" package="SO14" value="" x="-17.145" y="-24.765"/>
+<element name="U2" library="a_parts" package="SO14" value="" x="-17.145" y="-32.385"/>
+<element name="C2" library="a_parts" package="C0603" value="100n" x="-19.685" y="-38.1"/>
 </elements>
 <signals>
+<signal name="GND">
+<contactref element="U1" pad="11"/>
+<contactref element="U2" pad="11"/>
+<contactref element="C1" pad="2"/>
+<contactref element="C2" pad="2"/>
+<wire x1="-17.145" y1="-29.585" x2="-18.835" y2="-38.1" width="0" layer="19" extent="1-1"/>
+<wire x1="-17.145" y1="-21.965" x2="-17.145" y2="-29.585" width="0" layer="19" extent="1-1"/>
+<wire x1="9.105" y1="15.875" x2="-17.145" y2="-21.965" width="0" layer="19" extent="1-1"/>
+</signal>
+<signal name="3.3V">
+<contactref element="U1" pad="4"/>
+<contactref element="U2" pad="4"/>
+<contactref element="C1" pad="1"/>
+<contactref element="C2" pad="1"/>
+<wire x1="-17.145" y1="-35.185" x2="-20.535" y2="-38.1" width="0" layer="19" extent="1-1"/>
+<wire x1="-17.145" y1="-27.565" x2="-17.145" y2="-35.185" width="0" layer="19" extent="1-1"/>
+<wire x1="7.405" y1="15.875" x2="-17.145" y2="-27.565" width="0" layer="19" extent="1-1"/>
+</signal>
+<signal name="INA+">
+<contactref element="U1" pad="3"/>
+</signal>
+<signal name="INA-">
+<contactref element="U1" pad="2"/>
+</signal>
+<signal name="OUTC">
+<contactref element="U1" pad="8"/>
+</signal>
+<signal name="INB+">
+<contactref element="U1" pad="5"/>
+</signal>
+<signal name="INB-">
+<contactref element="U1" pad="6"/>
+</signal>
+<signal name="IND-">
+<contactref element="U1" pad="13"/>
+</signal>
+<signal name="IND+">
+<contactref element="U1" pad="12"/>
+</signal>
+<signal name="OUTB">
+<contactref element="U1" pad="7"/>
+</signal>
+<signal name="INC-">
+<contactref element="U1" pad="9"/>
+</signal>
+<signal name="INC+">
+<contactref element="U1" pad="10"/>
+</signal>
+<signal name="OUTA">
+<contactref element="U1" pad="1"/>
+</signal>
+<signal name="OUTD">
+<contactref element="U1" pad="14"/>
+</signal>
+<signal name="INE+">
+<contactref element="U2" pad="3"/>
+</signal>
+<signal name="INE-">
+<contactref element="U2" pad="2"/>
+</signal>
+<signal name="INF+">
+<contactref element="U2" pad="5"/>
+</signal>
+<signal name="INF-">
+<contactref element="U2" pad="6"/>
+</signal>
+<signal name="OUTH">
+<contactref element="U2" pad="14"/>
+</signal>
+<signal name="OUTG">
+<contactref element="U2" pad="8"/>
+</signal>
+<signal name="OUTE">
+<contactref element="U2" pad="1"/>
+</signal>
+<signal name="OUTF">
+<contactref element="U2" pad="7"/>
+</signal>
+<signal name="ING+">
+<contactref element="U2" pad="10"/>
+</signal>
+<signal name="ING-">
+<contactref element="U2" pad="9"/>
+</signal>
+<signal name="INH+">
+<contactref element="U2" pad="12"/>
+</signal>
+<signal name="INH-">
+<contactref element="U2" pad="13"/>
+</signal>
 </signals>
 </board>

Commit message: initial layout tomfoolery
Parts:
- added C10, C3, C4, C5, C6, C7, C8, C9: 100n, a_parts:C0603
- added JP1: M06JST-PH-PTH-VERT, a_parts:JST-6-PH-VERT-PTH
- added R1, R10, R13, R16, R19, R4, R7: 1K, a_parts:R0603
- added R11, R14, R17, R2, R20, R5, R8: 1M, a_parts:R0603
- added R12, R15, R18, R21, R3, R6, R9: 3K3, a_parts:R0603
- added U3: MCP3008, a_parts:SO16
- PD5: value GUVA-S12SD -> SD019-141-411-IR; device a_parts:LED3528 -> a_parts:LED-0805
- PD6: value GUVB-S11SD -> GUVA-S12SD
- PD7: value SD019-141-411-IR -> GUVB-S11SD; device a_parts:LED-0805 -> a_parts:LED3528
- U1, U2: value (none) -> MCP6004
- moved C2 83.5 mm to (40.6, 19.7)
- moved U2 73.3 mm to (40.6, 12.7), turned to 270 degrees
- moved PD7 64.1 mm to (33.0, 14.6), flipped to the bottom
- moved PD4 55.5 mm to (34.9, 9.53), flipped to the bottom, turned to 180 degrees
- moved U1 53.0 mm to (20.3, 12.7), turned to 270 degrees
- moved PD3 49.2 mm to (30.5, 9.53), flipped to the bottom, turned to 180 degrees
- moved PD5 46.4 mm to (39.4, 9.53), flipped to the bottom, turned to 180 degrees
- moved PD2 43.2 mm to (26.0, 9.53), flipped to the bottom, turned to 180 degrees
- moved PD1 37.8 mm to (21.6, 9.53), flipped to the bottom, turned to 180 degrees
- moved PD6 37.3 mm to (27.9, 14.6), flipped to the bottom
- moved C1 12.7 mm to (20.3, 19.7)
Connections:
- removed net INA+: U1.3
- removed net INB+: U1.5
- removed net INC+: U1.10
- removed net IND+: U1.12
- removed net INE+: U2.3
- removed net INF+: U2.5
- removed net ING+: U2.10
- removed net INH+: U2.12
- removed net INH-: U2.13
- removed net OUTH: U2.14
- new net !CS: JP1.6, U3.10
- new net MISO: JP1.4, U3.12
- new net MOSI: JP1.5, U3.11
- new net N$10: C7.1, R13.1, R14.2, R15.2
- new net N$11: C8.1, R16.1, R17.2, R18.2
- new net N$5: C3.1, R1.1, R2.2, R3.2
- new net N$6: C4.1, R4.1, R5.2, R6.2
- new net N$7: C5.1, R7.1, R8.2, R9.2
- new net N$8: C6.1, R10.1, R11.2, R12.2
- new net N$9: C9.1, R19.1, R20.2, R21.2
- new net SCK: JP1.3, U3.13
- net 3.3V: now also C10.1, JP1.1, U2.12, U3.15, U3.16
- net GND: now also C10.2, JP1.2, PD1.A, PD2.A, PD3.A, PD4.A, PD5.A, PD6.A, PD7.A, R1.2, R10.2, R13.2, R16.2, R19.2, R4.2, R7.2, U1.10, U1.12, U1.3, U1.5, U2.10, U2.13, U2.3, U2.5, U3.14, U3.9
- net INA-: now also C3.2, PD1.C, R2.1
- net INB-: now also C4.2, PD2.C, R5.1
- net INC-: now also C5.2, PD3.C, R8.1
- net IND-: now also C6.2, PD4.C, R11.1
- net INE-: now also C7.2, PD5.C, R14.1
- net INF-: now also C8.2, PD6.K, R17.1
- net ING-: now also C9.2, PD7.K, R20.1
- net OUTA: now also R3.1, U3.1
- net OUTB: now also R6.1, U3.2
- net OUTC: now also R9.1, U3.3
- net OUTD: now also R12.1, U3.4
- net OUTE: now also R15.1, U3.5
- net OUTF: now also R18.1, U3.6
- net OUTG: now also R21.1, U3.7
Routing:
- added copper zone on layer 1, net GND
- added copper zone on layer 16, net GND

Commit message: more photodiode dickery
Parts:
- moved C10 23.1 mm to (6.99, 28.6)
- moved U3 22.4 mm to (7.62, 34.9)
- moved C6 22.2 mm to (15.2, 13.3), turned to 90 degrees
- moved R16 19.1 mm to (30.5, 4.45), flipped to the bottom, turned to 90 degrees
- moved R11 18.8 mm to (17.8, 13.3), turned to 90 degrees
- moved C8 18.2 mm to (35.6, 4.45), turned to 90 degrees
- moved C2 18.2 mm to (26.0, 8.89), turned to 270 degrees
- moved R18 17.6 mm to (33.0, 4.45), flipped to the bottom, turned to 90 degrees
- moved C7 17.3 mm to (25.4, 13.3), turned to 90 degrees
- moved R17 17.3 mm to (38.1, 4.45), turned to 90 degrees
- moved PD5 14.0 mm to (25.4, 8.89), turned to 0 degrees
- moved R14 13.7 mm to (27.9, 13.3), turned to 90 degrees
- moved PD4 13.7 mm to (21.2, 10.0), turned to 90 degrees
- moved C4 13.1 mm to (13.0, 4.45), turned to 270 degrees
- moved R10 12.7 mm to (20.3, 13.3), flipped to the bottom, turned to 90 degrees
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Connections:
- net GND: now also R1.1, R10.1, R13.1, R16.1, R19.1, R4.1, R7.1; no longer R1.2, R10.2, R13.2, R16.2, R19.2, R4.2, R7.2
- net INA-: now also C3.1; no longer C3.2
- net INB-: now also C4.1; no longer C4.2
- net INC-: now also C5.1; no longer C5.2
- net IND-: now also C6.1; no longer C6.2
- net INE-: now also C7.1; no longer C7.2
- net INF-: now also C8.1; no longer C8.2
- net ING-: now also C9.1; no longer C9.2
- net N$10: now also C7.2, R13.2; no longer C7.1, R13.1
- net N$11: now also C8.2, R16.2; no longer C8.1, R16.1
- net N$5: now also C3.2, R1.2; no longer C3.1, R1.1
- net N$6: now also C4.2, R4.2; no longer C4.1, R4.1
- net N$7: now also C5.2, R7.2; no longer C5.1, R7.1
- net N$8: now also C6.2, R10.2; no longer C6.1, R10.1
- net N$9: now also C9.2, R19.2; no longer C9.1, R19.1
Other:
- board size 50.8 x 25.4 mm -> 50.8 x 17.8 mm
- board text added: "B"
- board text added: "C"
- board text added: "G"
- board text added: "IR"
- board text added: "R"
- board text added: "UVA"
- board text added: "UVB"
