File: hardware/tricorder-photodiode-breakout-mk-1.0.sch (EAGLE design)
At the start: 9 parts

Commit message: quad opamps
Parts:
- added C2: 100n, a_parts:CAPACITOR-CERAMICC0603
- added PD7: SD019-141-411-IR, a_parts:PHOTODIODESMD-0805
- added U2: (no value), a_parts:MCP6004SOIC14
- PD1: value GUVA-S12SD -> SD019-141-411-R; device a_parts:PHOTODIODESMD-3528 -> a_parts:PHOTODIODESMD-0805
- PD2: value GUVB-S11SD -> SD019-141-411-G; device a_parts:PHOTODIODESMD-3528 -> a_parts:PHOTODIODESMD-0805
- PD3: value SD019-141-411-R -> SD019-141-411-B
- PD4: value SD019-141-411-G -> SD019-111-411
- PD5: value SD019-141-411-B -> GUVA-S12SD; device a_parts:PHOTODIODESMD-0805 -> a_parts:PHOTODIODESMD-3528
- PD6: value SD019-111-411 -> GUVB-S11SD; device a_parts:PHOTODIODESMD-0805 -> a_parts:PHOTODIODESMD-3528
- U1: device a_parts:MCP6002SOIC -> a_parts:MCP6004SOIC14
Connections:
- new net 3.3V: C1.1, C2.1, U1.V+, U2.V+
- new net GND: C1.2, C2.2, U1.V-, U2.V-
- new net INA+: U1.INA+
- new net INA-: U1.INA-
- new net INB+: U1.INB+
- new net INB-: U1.INB-
- new net INC+: U1.INC+
- new net INC-: U1.INC-
- new net IND+: U1.IND+
- new net IND-: U1.IND-
- new net INE+: U2.INA+
- new net INE-: U2.INA-
- new net INF+: U2.INB+
- new net INF-: U2.INB-
- new net ING+: U2.INC+
- new net ING-: U2.INC-
- new net INH+: U2.IND+
- new net INH-: U2.IND-
- new net OUTA: U1.OUTA
- new net OUTB: U1.OUTB
- new net OUTC: U1.OUTC
- new net OUTD: U1.OUTD
- new net OUTE: U2.OUTA
- new net OUTF: U2.OUTB
- new net OUTG: U2.OUTC
- new net OUTH: U2.OUTD
Other:
- moved on the sheet: C1, PD1, PD2, PD3, PD4, PD5, PD6

Commit message: initial layout tomfoolery
Parts:
- added C10, C3, C4, C5, C6, C7, C8, C9: 100n, a_parts:CAPACITOR-CERAMICC0603
- added JP1: M06JST-PH-PTH-VERT, a_parts:M06JST-PH-PTH-VERT
- added R1, R10, R13, R16, R19, R4, R7: 1K, a_parts:RESISTORR0603
- added R11, R14, R17, R2, R20, R5, R8: 1M, a_parts:RESISTORR0603
- added R12, R15, R18, R21, R3, R6, R9: 3K3, a_parts:RESISTORR0603
- added U3: MCP3008, a_parts:MCP3008SOIC16
- PD5: value GUVA-S12SD -> SD019-141-411-IR; device a_parts:PHOTODIODESMD-3528 -> a_parts:PHOTODIODESMD-0805
- PD6: value GUVB-S11SD -> GUVA-S12SD
- PD7: value SD019-141-411-IR -> GUVB-S11SD; device a_parts:PHOTODIODESMD-0805 -> a_parts:PHOTODIODESMD-3528
- U1, U2: value (none) -> MCP6004
Connections:
- removed net INA+: U1.INA+
- removed net INB+: U1.INB+
- removed net INC+: U1.INC+
- removed net IND+: U1.IND+
- removed net INE+: U2.INA+
- removed net INF+: U2.INB+
- removed net ING+: U2.INC+
- removed net INH+: U2.IND+
- removed net INH-: U2.IND-
- removed net OUTH: U2.OUTD
- new net !CS: JP1.6, U3./CS
- new net MISO: JP1.4, U3.DOUT
- new net MOSI: JP1.5, U3.DIN
- new net N$10: C7.1, R13.1, R14.2, R15.2
- new net N$11: C8.1, R16.1, R17.2, R18.2
- new net N$5: C3.1, R1.1, R2.2, R3.2
- new net N$6: C4.1, R4.1, R5.2, R6.2
- new net N$7: C5.1, R7.1, R8.2, R9.2
- new net N$8: C6.1, R10.1, R11.2, R12.2
- new net N$9: C9.1, R19.1, R20.2, R21.2
- new net SCK: JP1.3, U3.CLK
- net 3.3V: now also C10.1, JP1.1, U2.IND+, U3.VDD, U3.VREF
- net GND: now also C10.2, JP1.2, PD1.A, PD2.A, PD3.A, PD4.A, PD5.A, PD6.A, PD7.A, R1.2, R10.2, R13.2, R16.2, R19.2, R4.2, R7.2, U1.INA+, U1.INB+, U1.INC+, U1.IND+, U2.INA+, U2.INB+, U2.INC+, U2.IND-, U3.AGND, U3.GND
- net INA-: now also C3.2, PD1.C, R2.1
- net INB-: now also C4.2, PD2.C, R5.1
- net INC-: now also C5.2, PD3.C, R8.1
- net IND-: now also C6.2, PD4.C, R11.1
- net INE-: now also C7.2, PD5.C, R14.1
- net INF-: now also C8.2, PD6.C, R17.1
- net ING-: now also C9.2, PD7.C, R20.1
- net OUTA: now also R3.1, U3.CH0
- net OUTB: now also R6.1, U3.CH1
- net OUTC: now also R9.1, U3.CH2
- net OUTD: now also R12.1, U3.CH3
- net OUTE: now also R15.1, U3.CH4
- net OUTF: now also R18.1, U3.CH5
- net OUTG: now also R21.1, U3.CH6
Other:
- moved on the sheet: C1, C2, PD1, PD2, PD3, PD4, PD5, PD6, PD7, U1, U2

Commit message: more photodiode dickery
Connections:
- net GND: now also R1.1, R10.1, R13.1, R16.1, R19.1, R4.1, R7.1; no longer R1.2, R10.2, R13.2, R16.2, R19.2, R4.2, R7.2
- net INA-: now also C3.1; no longer C3.2
- net INB-: now also C4.1; no longer C4.2
- net INC-: now also C5.1; no longer C5.2
- net IND-: now also C6.1; no longer C6.2
- net INE-: now also C7.1; no longer C7.2
- net INF-: now also C8.1; no longer C8.2
- net ING-: now also C9.1; no longer C9.2
- net N$10: now also C7.2, R13.2; no longer C7.1, R13.1
- net N$11: now also C8.2, R16.2; no longer C8.1, R16.1
- net N$5: now also C3.2, R1.2; no longer C3.1, R1.1
- net N$6: now also C4.2, R4.2; no longer C4.1, R4.1
- net N$7: now also C5.2, R7.2; no longer C5.1, R7.1
- net N$8: now also C6.2, R10.2; no longer C6.1, R10.1
- net N$9: now also C9.2, R19.2; no longer C9.1, R19.1
Other:
- note added: "BLUE"
- note added: "CLEAR"
- note added: "GREEN"
- note added: "IR"
- note added: "RED"
- note added: "UVA"
- note added: "UVB"
- moved on the sheet: C3, C4, C5, C6, C7, C8, C9, R1, R10, R13, R16, R19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
