File: hardware/tricorder-featherwing-mk-1.0.sch (EAGLE design)
At the start: 7 parts, among them U1 ADAFRUIT_FEATHER_SHIELDSMALLH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

Commit message: connector board markup?
Parts:
- removed J$1: SMA_EDGE, a_parts:SMA_EDGE
- removed JP1: M10PTH, a_parts:M10PTH
- removed JP2: M04PTH, a_parts:M04PTH
- removed JP3: M05X2PTH, a_parts:M05X2PTH
- removed U2: (no value), a_parts:GPS_FGPMMOPA6H
- added C1: 10uF, a_parts:CAPACITOR-CERAMICC1210
- added C2: 1uF, a_parts:CAPACITOR-CERAMICC0603
- added DISPLAY: M05X2PTH, a_parts:M05X2PTH
- added FEATHERWING: ADAFRUIT_FEATHER_SHIELDSMALLHOLES_NS, a_parts:ADAFRUIT_FEATHER_SHIELDSMALLHOLES_NS
- added GPS_ANT: (no value), a_parts:ANTENNA_U.FL
- added GPS_RX, GPS_TX: (no value), a_parts:JUMPER-PAD-3-NOFULL_BOX_SILK
- added I2C: M04PTH, a_parts:M04PTH
- U1: value ADAFRUIT_FEATHER_SHIELDSMALLHOLES_NS -> (none); device a_parts:ADAFRUIT_FEATHER_SHIELDSMALLHOLES_NS -> a_parts:GPS_FGPMMOPA6H
Connections:
- new net 3.3V: C1.1, C2.1, DISPLAY.9, FEATHERWING.3V, I2C.2, U1.VCC
- new net DISP_CS: DISPLAY.5, FEATHERWING.10
- new net DISP_DC: DISPLAY.3, FEATHERWING.9
- new net DISP_RST: DISPLAY.4, FEATHERWING.A5
- new net GND: C1.2, C2.2, DISPLAY.10, FEATHERWING.GND, GPS_ANT.GND@0, GPS_ANT.GND@1, I2C.1, U1.GND@1, U1.GND@2, U1.GND@3, U1.GND@4
- new net GPS_RX: GPS_RX.2, U1.RX
- new net GPS_RX1: FEATHERWING.6, GPS_RX.1
- new net GPS_RX2: FEATHERWING.13, GPS_RX.3
- new net GPS_TX: GPS_TX.2, U1.TX
- new net GPS_TX1: FEATHERWING.5, GPS_TX.3
- new net GPS_TX2: FEATHERWING.12, GPS_TX.1
- new net MISO: DISPLAY.7, FEATHERWING.MISO
- new net MOSI: DISPLAY.1, FEATHERWING.MOSI
- new net SCK: DISPLAY.2, FEATHERWING.SCK
- new net SCL: FEATHERWING.SCL, I2C.3
- new net SDA: FEATHERWING.SDA, I2C.4
- new net SD_CS: DISPLAY.6, FEATHERWING.A4
- new net SD_SW: DISPLAY.8, FEATHERWING.A3
- net N$1: now also GPS_ANT.SIGNAL, U1.EX_ANT; no longer J$1.SIGNAL, U2.EX_ANT
