File: hardware/tricorder-featherwing-mk-1.3.sch (EAGLE design)
At the start: 7 parts

Commit message: jst version off to fab
Parts:
- added C3: 10uF, a_parts:CAPACITOR-CERAMICC1210
- I2C: value M04-I2CJST-4-PH-RA-CENTERED -> M04-I2CPTH-0.1IN-CENTERED; device a_parts:M04-I2CJST-4-PH-RA-CENTERED -> a_parts:M04-I2CPTH-0.1IN-CENTERED
- renumbered U1 to GPS
Connections:
- net 3.3V: now also C3.1, DISP/MICROSD.9
- net DISP_CS: now also DISP/MICROSD.5, FEATHERWING.A3; no longer FEATHERWING.11
- net DISP_DC: now also DISP/MICROSD.3, FEATHERWING.A1; no longer FEATHERWING.10
- net DISP_RST: now also DISP/MICROSD.4, FEATHERWING.A2; no longer FEATHERWING.A5
- net GND: now also C3.2, DISP/MICROSD.10
- net GPS_RX: now also FEATHERWING.12
- net GPS_TX: now also FEATHERWING.13
- net MISO: now also DISP/MICROSD.7
- net MOSI: now also DISP/MICROSD.1
- net SCK: now also DISP/MICROSD.2
- net SD_CS: now also DISP/MICROSD.6
- net SD_SW: now also DISP/MICROSD.8, FEATHERWING.A5; no longer FEATHERWING.A3
