File: hardware/gps-breakout-mk-1.1.brd (EAGLE design)
At the start: 16.5 x 21 mm, 4 parts

Commit message: first revision on gps module board
Parts:
- added ANT: (no value), a_parts:U.FL
- C1: device a_parts:C0603 -> a_parts:C0402
- moved JP1 2.93 mm to (8.26, 1.27)
- moved C1 1.37 mm to (1.91, 1.91)
- moved GPS 0.63 mm to (8.26, 11.4)
Connections:
- new net N$1: ANT.3, GPS.P$11
- net GND: now also ANT.1, ANT.2
Routing:
- net GND: track 13.2 -> 23.7 mm
- net GPS_TX: track 3.48 -> 7.88 mm, vias 0 -> 1
- net N$1: track 0.00 -> 2.74 mm, vias 0 -> 1
- net GPS_RX: track 3.05 -> 4.99 mm
- net 3.3V: track 8.64 -> 9.89 mm, vias 0 -> 1
Other:
- board size 16.5 x 21 mm -> 16.5 x 20.3 mm
- board text added: "+"
- board text added: "-"
- board text removed: "GND"
- board text removed: "VCC"
