File: hardware/gps-breakout-mk-1.1.sch (EAGLE design)
At the start: 4 parts

Commit message: first revision on gps module board
Parts:
- added ANT: (no value), a_parts:ANTENNA_U.FL
- C1: device a_parts:CAPACITOR-CERAMICC0603 -> a_parts:CAPACITOR-CERAMICC0402
Connections:
- new net N$1: ANT.SIGNAL, GPS.EX_ANT
- net GND: now also ANT.GND@0, ANT.GND@1
Changed lines of the file:
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@@
 <part name="GND6" library="a_parts" deviceset="GND" device=""/>
 <part name="SUPPLY5" library="a_parts" deviceset="3.3V" device=""/>
-<part name="C1" library="a_parts" deviceset="CAPACITOR-CERAMIC" device="C0603" value="1uF"/>
+<part name="C1" library="a_parts" deviceset="CAPACITOR-CERAMIC" device="C0402" value="1uF"/>
 <part name="SUPPLY7" library="a_parts" deviceset="3.3V" device=""/>
 <part name="GND8" library="a_parts" deviceset="GND" device=""/>
@@
 <part name="GND1" library="a_parts" deviceset="GND" device=""/>
 <part name="JP1" library="a_parts" deviceset="M04" device="PTH-NS-CENTERED" value="M04PTH-NS-CENTERED"/>
+<part name="ANT" library="a_parts" deviceset="ANTENNA_U.FL" device=""/>
 </parts>
 <sheets>
@@
 <instance part="GND1" gate="1" x="66.04" y="147.32"/>
 <instance part="JP1" gate="G$1" x="45.72" y="149.86"/>
+<instance part="ANT" gate="G$1" x="182.88" y="119.38" rot="R90"/>
 </instances>
 <busses>
@@
 <wire x1="193.04" y1="147.32" x2="193.04" y2="129.54" width="0.1524" layer="91"/>
 <junction x="193.04" y="129.54"/>
-<wire x1="132.08" y1="114.3" x2="193.04" y2="114.3" width="0.1524" layer="91"/>
+<wire x1="132.08" y1="114.3" x2="187.96" y2="114.3" width="0.1524" layer="91"/>
 <junction x="132.08" y="114.3"/>
+<pinref part="ANT" gate="G$1" pin="GND@0"/>
+<wire x1="187.96" y1="114.3" x2="190.5" y2="114.3" width="0.1524" layer="91"/>
+<wire x1="190.5" y1="114.3" x2="193.04" y2="114.3" width="0.1524" layer="91"/>
+<wire x1="187.96" y1="116.84" x2="187.96" y2="114.3" width="0.1524" layer="91"/>
+<junction x="187.96" y="114.3"/>
+<pinref part="ANT" gate="G$1" pin="GND@1"/>
+<wire x1="190.5" y1="116.84" x2="190.5" y2="114.3" width="0.1524" layer="91"/>
+<junction x="190.5" y="114.3"/>
 </segment>
 <segment>
@@
 </segment>
 </net>
+<net name="N$1" class="0">
+<segment>
+<pinref part="GPS" gate="G$1" pin="EX_ANT"/>
+<wire x1="177.8" y1="127" x2="182.88" y2="127" width="0.1524" layer="91"/>
+<pinref part="ANT" gate="G$1" pin="SIGNAL"/>
+<wire x1="182.88" y1="127" x2="182.88" y2="124.46" width="0.1524" layer="91"/>
+</segment>
+</net>
