File: hardware/tricorder-teensy-mk-1.0.brd (EAGLE design)
At the start: 49.5 x 24.1 mm, 23 parts, among them IC1 MCP73831, J1 TEENSY-3.1SMT_BOTTOM, U1 MICS-6814

Commit message: wip teensy hat layout
Parts:
- removed CHG: LED0603-TIGHT, a_parts:LED-0603-TIGHT
- removed D1: PMEG2005, a_parts:SOT23
- removed IC1: MCP73831, a_parts:SOT95P280X145-5N
- added CHARGING: LED0603-TIGHT, a_parts:LED-0603-TIGHT
- added D2: (no value), a_parts:SOD323-SCHOTTKY
- added GAS: M04SMD_RA_2MM, a_parts:1X04_SMD_RA_2MM
- added GAS_V: (no value), a_parts:PAD-JUMPER-3-NO_YES_SILK_FULL_BOX
- C3: value 10uF -> 4u7; device a_parts:C0805-TIGHTER -> a_parts:C0603-TIGHTER
- R3: value 1K -> 2K
- R4: value 2K -> 100k
- R6: value 100k -> 1K
- U1: value MICS-6814 -> MCP73831; device a_parts:MICS-10-PIN -> a_parts:SOT95P280X145-5N
- moved R2 35.3 mm to (19.1, 11.4), flipped to the bottom
- moved U1 35.2 mm to (60.3, 21.0), turned to 180 degrees
- moved R1 34.7 mm to (21.6, 11.4), flipped to the bottom
- moved R6 25.3 mm to (61.6, 15.9), flipped to the top, turned to 90 degrees
- moved C1 23.6 mm to (27.9, 11.4), turned to 90 degrees
- moved C2 20.7 mm to (64.1, 21.0), flipped to the top
- moved BATT 13.4 mm to (43.8, 5.71), turned to 180 degrees
- moved R3 12.1 mm to (54.0, 16.0), turned to 90 degrees
- moved R4 11.3 mm to (56.5, 15.9), turned to 90 degrees
- moved C3 9.71 mm to (54.0, 21.0), turned to 270 degrees
- moved R5 8.28 mm to (59.1, 15.9), turned to 270 degrees
- moved PROG 5.72 mm to (1.91, 12.1)
- moved J8 2.62 mm to (22.9, 4.45), turned to 270 degrees
- moved J7 2.01 mm to (20.3, 4.45), turned to 270 degrees
- moved GPS 0.63 mm to (8.89, 12.1)
- renumbered J1 to TEENSY
Connections:
- new net GAS_ANALOG: GAS.3, TEENSY.21/A7
- new net GAS_EN: GAS.4, TEENSY.9
- new net N$3: GAS.1, GAS_V.2
- net 3.3V: now also GAS_V.3
- net BATT_DIV: now also R4.1, R5.2; no longer R5.1, R6.2
- net GND: now also GAS.2, R3.1, R5.1, U1.2; no longer IC1.2, R4.1, R6.1
- net N$1: now also R6.2, U1.1; no longer CHG.C, IC1.1
- net N$2: now also CHARGING.C, R6.1; no longer CHG.A, R3.2
- net N$4: now also R3.2, U1.5; no longer IC1.5, R4.2
- net VBAT: now also D2.A, R4.2, U1.3; no longer D1.2, IC1.3, R5.2
- net VUSB: now also CHARGING.A, D2.C, GAS_V.1, U1.4; no longer D1.3, IC1.4, R3.1
Other:
- board text added: "GPS RX"
- board text added: "GPS TX"
