File: hardware/tricorder-teensy-mk-1.0.sch (EAGLE design)
At the start: 22 parts, among them IC1 MCP73831, J1 TEENSY-3.1SMT_BOTTOM, U1 MICS-6814

Commit message: wip teensy hat layout
Parts:
- removed CHG: LED0603-TIGHT, a_parts:LED0603-TIGHT
- removed D1: PMEG2005, a_parts:DIODE-SCHOTTKY-DUALPMEG2005CT
- removed IC1: MCP73831, a_parts:MCP73831T-2ACI/OT
- added CHARGING: LED0603-TIGHT, a_parts:LED0603-TIGHT
- added D2: (no value), a_parts:DIODE-SCHOTTKYSOD323
- added GAS: M04SMD_RA_2MM, a_parts:M04SMD_RA_2MM
- added GAS_V: (no value), a_parts:JUMPER-PAD-3-NOFULL_BOX_SILK
- C3: value 10uF -> 4u7; device a_parts:CAPACITOR-CERAMICC0805-TIGHTER -> a_parts:CAPACITOR-CERAMICC0603-TIGHTER
- R3: value 1K -> 2K
- R4: value 2K -> 100k
- R6: value 100k -> 1K
- U1: value MICS-6814 -> MCP73831; device a_parts:MICS-6814 -> a_parts:MCP73831T-2ACI/OT
- renumbered J1 to TEENSY
Connections:
- new net GAS_ANALOG: GAS.3, TEENSY.A7/21*
- new net GAS_EN: GAS.4, TEENSY.9*/RX2
- new net N$3: GAS.1, GAS_V.2
- net 3.3V: now also GAS_V.3
- net BATT_DIV: now also R4.1, R5.2; no longer R5.1, R6.2
- net GND: now also GAS.2, R3.1, R5.1, U1.VSS; no longer IC1.VSS, R4.1, R6.1
- net N$1: now also R6.2, U1.STAT; no longer CHG.C, IC1.STAT
- net N$2: now also CHARGING.C, R6.1; no longer CHG.A, R3.2
- net N$4: now also R3.2, U1.PROG; no longer IC1.PROG, R4.2
- net VBAT: now also D2.A, R4.2, U1.VBAT; no longer D1.A2, IC1.VBAT, R5.2
- net VUSB: now also CHARGING.A, D2.C, GAS_V.1, U1.VDD; no longer D1.K, IC1.VDD, R3.1
Other:
- moved on the sheet: R3, R4, R5, R6
