File: hardware/tricorder-teensy-mk-1.10.sch (EAGLE design)
At the start: 23 parts, among them U1 MCP73831, U2 LTC2941

Commit message: layout complete
Parts:
- D1: value (none) -> MBRS0540
Connections:
- net !AL/CC: now also TEENSY.A14/DAC; no longer TEENSY.2
Other:
- moved on the sheet: D1
Changed lines of the file:
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@@
 <part name="GND11" library="a_parts" deviceset="GND" device=""/>
 <part name="GND1" library="a_parts" deviceset="GND" device=""/>
-<part name="D1" library="a_parts" deviceset="DIODE-SCHOTTKY" device="SOD123"/>
+<part name="D1" library="a_parts" deviceset="DIODE-SCHOTTKY" device="SOD123" value="MBRS0540"/>
 <part name="PWR_SW" library="a_parts" deviceset="M02" device="JST-2MM-SMT"/>
 <part name="GPS_RX_ALT" library="a_parts" deviceset="JUMPER-PAD-3-NO" device="FULL_BOX_SILK"/>
@@
 <instance part="SUPPLY15" gate="G$1" x="195.58" y="83.82"/>
 <instance part="C2" gate="G$1" x="195.58" y="73.66"/>
-<instance part="SUPPLY7" gate="G$1" x="218.44" y="83.82"/>
+<instance part="SUPPLY7" gate="G$1" x="220.98" y="83.82"/>
 <instance part="C3" gate="G$1" x="17.78" y="129.54"/>
 <instance part="SUPPLY9" gate="G$1" x="17.78" y="139.7"/>
 <instance part="GND11" gate="1" x="17.78" y="116.84"/>
 <instance part="GND1" gate="1" x="38.1" y="149.86"/>
-<instance part="D1" gate="G$1" x="205.74" y="81.28"/>
+<instance part="D1" gate="G$1" x="208.28" y="81.28"/>
 <instance part="PWR_SW" gate="G$1" x="15.24" y="50.8"/>
 <instance part="GPS_RX_ALT" gate="G$1" x="226.06" y="142.24"/>
@@
 <wire x1="195.58" y1="81.28" x2="185.42" y2="81.28" width="0.1524" layer="91"/>
 <junction x="195.58" y="81.28"/>
-<wire x1="195.58" y1="81.28" x2="203.2" y2="81.28" width="0.1524" layer="91"/>
+<wire x1="195.58" y1="81.28" x2="205.74" y2="81.28" width="0.1524" layer="91"/>
 <pinref part="D1" gate="G$1" pin="A"/>
 </segment>
@@
 </segment>
 <segment>
-<wire x1="208.28" y1="81.28" x2="218.44" y2="81.28" width="0.1524" layer="91"/>
+<wire x1="210.82" y1="81.28" x2="220.98" y2="81.28" width="0.1524" layer="91"/>
 <pinref part="SUPPLY7" gate="G$1" pin="VUSB"/>
-<wire x1="218.44" y1="81.28" x2="218.44" y2="83.82" width="0.1524" layer="91"/>
+<wire x1="220.98" y1="81.28" x2="220.98" y2="83.82" width="0.1524" layer="91"/>
 <pinref part="D1" gate="G$1" pin="C"/>
 </segment>
@@
 </segment>
 <segment>
-<pinref part="TEENSY" gate="G$1" pin="2"/>
-<wire x1="190.5" y1="147.32" x2="185.42" y2="147.32" width="0.1524" layer="91"/>
-<label x="190.5" y="147.32" size="1.27" layer="95" xref="yes"/>
-</segment>
-</net>
+<wire x1="144.78" y1="142.24" x2="149.86" y2="142.24" width="0.1524" layer="91"/>
+<label x="144.78" y="142.24" size="1.27" layer="95" rot="R180" xref="yes"/>
+<pinref part="TEENSY" gate="G$1" pin="A14/DAC"/>
+</segment>
+</net>
