File: hardware/tricorder-teensy-mk-1.10.brd (EAGLE design)
At the start: 50.8 x 22.9 mm, 23 parts, among them U1 MCP73831, U2 LTC2941

Commit message: layout complete
Parts:
- added U$1: (no value), a_parts:COW
- D1: value (none) -> MBRS0540
- moved CHRG 15.9 mm to (44.5, 3.17), turned to 270 degrees
- moved R2 13.1 mm to (11.4, 14.6), turned to 0 degrees
- moved R1 12.7 mm to (14.0, 12.1), turned to 0 degrees
- moved R6 10.8 mm to (41.9, 3.17), turned to 270 degrees
- moved C2 4.45 mm to (39.4, 3.17)
- moved C3 4.45 mm to (31.8, 3.17)
- moved R3 4.45 mm to (29.2, 3.17)
- moved U1 4.45 mm to (35.6, 3.17)
- moved D1 1.27 mm to (35.6, 6.99)
Connections:
- net !AL/CC: now also TEENSY.A14/DAC; no longer TEENSY.2
Routing:
- net 3.3V: track 0.00 -> 69.2 mm, vias 0 -> 2
- net VUSB: track 0.00 -> 61.1 mm, vias 0 -> 3
- net SCL: track 11.4 -> 57.1 mm, vias 0 -> 1
- net PROG: track 0.00 -> 39.7 mm, vias 0 -> 2
- net SDA: track 6.98 -> 46.3 mm, vias 0 -> 1
- net GPS_TX: track 0.00 -> 32.3 mm, vias 0 -> 2
- net GPS_RX: track 0.00 -> 28.5 mm, vias 0 -> 2
- net !AL/CC: track 0.00 -> 21.6 mm, vias 0 -> 1
- net SD_SW: track 0.00 -> 21.1 mm, vias 0 -> 1
- net SCK: track 0.00 -> 19.6 mm, vias 0 -> 1
- net MOSI: track 0.00 -> 18.0 mm, vias 0 -> 1
- net VBAT: track 3.44 -> 18.7 mm
- net MISO: track 0.00 -> 14.8 mm, vias 0 -> 1
- net 8/TX3: track 0.00 -> 14.8 mm
- net !DISP_CS: track 0.00 -> 12.8 mm, vias 0 -> 1
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Other:
- board text added: "by sean@yak.net CC-4.0-BY-SA"

Commit message: silkscreen fix because of course
Parts:
- U$1: device a_parts:COW -> a_parts:COW_SMALL
- moved U$1 3.30 mm to (8.89, 16.0)
Changed lines of the file:
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@@
 </element>
 <element name="C1" library="a_parts" package="C1210" value="10uF" x="36.83" y="10.16" smashed="yes" rot="R180">
-<attribute name="NAME" x="34.29" y="10.16" size="0.8128" layer="25" font="vector" ratio="10" rot="R90" align="bottom-center"/>
-<attribute name="VALUE" x="39.37" y="10.16" size="0.6096" layer="27" font="vector" ratio="10" rot="R90" align="top-center"/>
+<attribute name="NAME" x="34.163" y="10.16" size="0.8128" layer="25" font="vector" ratio="10" rot="R90" align="bottom-center"/>
+<attribute name="VALUE" x="39.497" y="10.16" size="0.6096" layer="21" font="vector" ratio="10" rot="R90" align="top-center"/>
 </element>
 <element name="I2C" library="a_parts" package="1X04_SMD_RA_2MM_I2C" value="M04-I2CSMD_2MM_RA" x="43.18" y="14.605" smashed="yes">
-<attribute name="NAME" x="43.18" y="12.573" size="1.016" layer="25" font="vector" ratio="10" align="top-center"/>
+<attribute name="NAME" x="43.18" y="12.446" size="1.016" layer="25" font="vector" ratio="10" align="top-center"/>
 </element>
 <element name="DISPLAY" library="a_parts" package="1X10_SMD_RA_MALE" value="M10SMD_RA_2MM" x="28.575" y="14.605" smashed="yes">
-<attribute name="NAME" x="28.542" y="12.565" size="1.016" layer="25" font="vector" ratio="10" align="top-center"/>
+<attribute name="NAME" x="28.542" y="12.438" size="1.016" layer="25" font="vector" ratio="10" align="top-center"/>
 </element>
 <element name="R1" library="a_parts" package="R0603-TIGHTER" value="4K7" x="13.97" y="12.065" smashed="yes" rot="MR0">
@@
 <attribute name="OC_FARNELL" value="1332158" x="35.56" y="3.175" size="1.778" layer="27" rot="R180" display="off"/>
 <attribute name="NAME" x="35.56" y="4.925" size="0.8128" layer="25" font="vector" ratio="10" rot="SR0" align="bottom-center"/>
-<attribute name="VALUE" x="35.56" y="1.425" size="0.6096" layer="27" font="vector" ratio="10" rot="R180" align="bottom-center"/>
+<attribute name="VALUE" x="35.56" y="1.425" size="0.6096" layer="21" font="vector" ratio="10" rot="R180" align="bottom-center"/>
 </element>
 <element name="CHRG" library="a_parts" package="LED-0603-TIGHT" value="LED0603-TIGHT" x="44.45" y="3.175" smashed="yes" rot="R270">
@@
 <element name="R6" library="a_parts" package="R0603-TIGHTER" value="1K" x="41.91" y="3.175" smashed="yes" rot="R270">
 <attribute name="NAME" x="41.91" y="4.826" size="0.8128" layer="25" font="vector" ratio="10" align="bottom-center"/>
-<attribute name="VALUE" x="41.91" y="1.625" size="0.6096" layer="25" font="vector" ratio="10" align="top-center"/>
+<attribute name="VALUE" x="41.91" y="1.498" size="0.6096" layer="25" font="vector" ratio="10" align="top-center"/>
 </element>
 <element name="R3" library="a_parts" package="R0603-TIGHTER" value="2K" x="29.21" y="3.175" smashed="yes" rot="R270">
 <attribute name="NAME" x="29.21" y="4.826" size="0.8128" layer="25" font="vector" ratio="10" align="bottom-center"/>
-<attribute name="VALUE" x="29.21" y="1.625" size="0.6096" layer="25" font="vector" ratio="10" align="top-center"/>
+<attribute name="VALUE" x="29.21" y="1.498" size="0.6096" layer="25" font="vector" ratio="10" align="top-center"/>
 </element>
 <element name="C2" library="a_parts" package="C0603-TIGHTER" value="4u7" x="39.37" y="3.175" smashed="yes" rot="R270">
 <attribute name="NAME" x="39.37" y="4.826" size="0.8128" layer="25" font="vector" ratio="10" align="bottom-center"/>
-<attribute name="VALUE" x="39.37" y="1.651" size="0.6096" layer="25" font="vector" ratio="10" align="top-center"/>
+<attribute name="VALUE" x="39.37" y="1.524" size="0.6096" layer="25" font="vector" ratio="10" align="top-center"/>
 </element>
 <element name="C3" library="a_parts" package="C0603-TIGHTER" value="4u7" x="31.75" y="3.175" smashed="yes" rot="R270">
 <attribute name="NAME" x="31.75" y="4.826" size="0.8128" layer="25" font="vector" ratio="10" align="bottom-center"/>
-<attribute name="VALUE" x="31.75" y="1.651" size="0.6096" layer="25" font="vector" ratio="10" align="top-center"/>
+<attribute name="VALUE" x="31.75" y="1.524" size="0.6096" layer="25" font="vector" ratio="10" align="top-center"/>
 </element>
 <element name="D1" library="a_parts" package="SOD123-SCHOTTKY" value="MBRS0540" x="35.56" y="6.985" smashed="yes" rot="R180">
@@
 <element name="U2" library="a_parts" package="MSOP-8" value="LTC2941" x="47.625" y="8.255" smashed="yes" rot="R90">
 <attribute name="NAME" x="45.925" y="8.255" size="0.8128" layer="25" font="vector" ratio="10" rot="R90" align="bottom-center"/>
-<attribute name="VALUE" x="49.325" y="8.255" size="0.6096" layer="27" font="vector" ratio="10" rot="R90" align="top-center"/>
+<attribute name="VALUE" x="49.452" y="8.255" size="0.6096" layer="21" font="vector" ratio="10" rot="R90" align="top-center"/>
 </element>
 <element name="R4" library="a_parts" package="R0603-TIGHTER" value="0R1" x="43.815" y="8.255" smashed="yes" rot="R270">
 <attribute name="NAME" x="43.815" y="9.779" size="0.8128" layer="25" font="vector" ratio="10" align="bottom-center"/>
-<attribute name="VALUE" x="43.815" y="6.731" size="0.6096" layer="27" font="vector" ratio="10" align="top-center"/>
+<attribute name="VALUE" x="43.815" y="6.604" size="0.6096" layer="21" font="vector" ratio="10" align="top-center"/>
 </element>
 <element name="C4" library="a_parts" package="C0603-TIGHTER" value="100n" x="41.275" y="8.255" smashed="yes" rot="R90">
 <attribute name="NAME" x="41.275" y="9.779" size="0.8128" layer="25" font="vector" ratio="10" align="bottom-center"/>
-<attribute name="VALUE" x="41.275" y="6.705" size="0.6096" layer="27" font="vector" ratio="10" align="top-center"/>
+<attribute name="VALUE" x="41.275" y="6.578" size="0.6096" layer="21" font="vector" ratio="10" align="top-center"/>
 </element>
-<element name="U$1" library="a_parts" package="COW" value="" x="8.89" y="12.7"/>
+<element name="U$1" library="a_parts" package="COW_SMALL" value="" x="8.89" y="16.002"/>
 </elements>
 <signals>
