File: hardware/tricorder-teensy-mk-1.11.sch (EAGLE design)
At the start: 23 parts, among them U1 MCP73831, U2 LTC2941

Commit message: new revision with LTC2942 instead of '41
Parts:
- added C5: 100n, a_parts:CAPACITOR-CERAMICC0603-TIGHTER
- C1: value 10uF -> 100uF
- GPS_RX_ALT, GPS_TX_ALT: value (none) -> JUMPER-PAD-3-NOFULL_BOX_SILK
- R4: device a_parts:RESISTORR0603-TIGHTER -> a_parts:RESISTORR0805-TIGHTER
- TEENSY: value TEENSY-3.1-OUTERSMT -> TEENSY-3.1-OUTERSMD; device a_parts:TEENSY-3.1-OUTERSMT -> a_parts:TEENSY-3.1-OUTERSMD
- U2: device a_parts:LTC2941MSOP-8 -> a_parts:LTC2941/2DCB
Connections:
- net N$1 renamed STAT
- net N$2 renamed CHARGING
- net N$3 renamed BEFORE_SW
- net N$4 renamed CURRENT_SET
- net N$5 renamed AFTER_SW
- net 3.3V: now also C1.2, C5.1; no longer C1.1
- net GND: now also C1.1, C5.2; no longer C1.2
Other:
- moved on the sheet: C1
